File: mac_paddy/mac_paddy.kicad_sch (KiCad schematic)
At the start: 13 parts, among them SW1 SW_Push, SW2 SW_Push, SW3 SW_Push, SW4 SW_Push, SW5 SW_Push, SW6 SW_Push, U1 XIAO-ESP32-S3-SMD

Commit message: PCB design and export completed!
Parts:
- added D10, D11, D12, D7, D8, D9: WS2812B, LED_SMD:LED_WS2812B_PLCC4_5.0x5.0mm_P3.2mm, symbol LED:WS2812B
- added D13: 1N4148, ScottoKeebs_Components:Diode_DO-35, symbol Diode:1N4148
- added J1: OLED_128x32, ScottoKeebs_Components:OLED_128x32, symbol ScottoKeebs:OLED_128x32
- added SW7: RotaryEncoder_Switch, ScottoKeebs_Scotto:Encoder_EC11_MX, symbol Device:RotaryEncoder_Switch
Connections:
- net ROW 1: now also D13.1 (K)
- net GND: now reaches U1.13 (GND)
- net GND: now also D10.3 (VSS), D11.3 (VSS), D12.3 (VSS), D7.3 (VSS), D8.3 (VSS), D9.3 (VSS), J1.1 (GND), SW7.C
- net VCC: now reaches U1.14 (VBUS)
- net VCC: now also D10.1 (VDD), D11.1 (VDD), D12.1 (VDD), D7.1 (VDD), D8.1 (VDD), D9.1 (VDD), J1.2 (VCC)
- net LED-IN: now reaches U1.4 (GPIO4_A3_D3)
- net LED-IN: now also D7.4 (DIN)
- net OLED-SDA: now reaches U1.5 (GPIO5_A4_D4_SDA)
- net OLED-SDA: now also J1.4 (SDA)
- net OLED-SCL: now reaches U1.6 (GPIO6_A5_D5_SCL)
- net OLED-SCL: now also J1.3 (SCL)
- net ENC-S1: now reaches U1.7 (GPIO43_D6_TX)
- net ENC-S1: now also SW7.S1
- net ENC-B: now reaches U1.8 (GPIO44_D7_RX)
- net ENC-B: now also SW7.B
- net ENC-A: now reaches U1.9 (GPIO7_A8_D8_SCK)
- net ENC-A: now also SW7.A
- new net: D10.4 (DIN), D9.2 (DOUT)
- new net: D8.2 (DOUT), D9.4 (DIN)
- new net: D7.2 (DOUT), D8.4 (DIN)
- new net: D10.2 (DOUT), D11.4 (DIN)
- new net: D13.2 (A), SW7.S2
- new net: D11.2 (DOUT), D12.4 (DIN)
- no-connect marks 20 -> 13
Other:
- note added: "LED DAISY CHAIN"
- note added: "OLED SCREEN"
- note added: "ROTARY ENCODER"
- note added: "SWITCH MATRIX"
- moved on the sheet: D1, D2, D3, D4, D5, D6, SW1, SW2, SW3, SW4, SW5, SW6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
